File: hardware/deflection_amp/deflection_amp.kicad_sch (KiCad schematic)
At the start: 41 parts, among them U1 6SN7, U2 6SN7, U3 6SN7

Commit message: Draft deflection amp pcb done
Parts:
- removed C1, C2: 16uF, symbol Device:C
- removed J?: Conn_01x04, symbol Connector_Generic:Conn_01x04
- added C1: 10uF 500V, Capacitor_THT:CP_Radial_D12.5mm_P5.00mm, symbol Device:C_Polarized_US
- added H1, H2, H3, H4: MTG, MountingHole:MountingHole_4.5mm_Pad, symbol Mechanical:MountingHole_Pad
- added J3: Conn_01x03, Connector_Molex:Molex_KK-396_A-41791-0003_1x03_P3.96mm_Vertical, symbol Connector_Generic:Conn_01x03
- C10, C9: footprint (none) -> Capacitor_THT:C_Disc_D3.8mm_W2.6mm_P2.50mm; CatNo (none) -> 399-14010-2-ND
- C3, C4: footprint (none) -> HV_Ceramic_Cap:Cap-Disc-D7.4-P6.4; CatNo (none) -> 561R10TCCQ25-ND
- C5, C6: value 2uF -> 2.2uF 250V; footprint (none) -> Capacitor_THT:C_Rect_L26.5mm_W8.5mm_P22.50mm_MKS4; CatNo (none) -> EF2225-ND
- C7, C8: footprint (none) -> Capacitor_THT:C_Disc_D8.0mm_W2.5mm_P5.00mm; CatNo (none) -> 445-173352-1-ND
- J1: renamed from J?; footprint (none) -> Connector_Molex:Molex_KK-396_A-41791-0002_1x02_P3.96mm_Vertical
- J2: renamed from J?; footprint (none) -> Connector_PinHeader_2.54mm:PinHeader_1x04_P2.54mm_Vertical
- J4: renamed from J?; footprint (none) -> Connector_PinHeader_2.54mm:PinHeader_1x06_P2.54mm_Vertical
- R1, R19, R2, R21, R7, R9: value 1M -> 1M 1/2W; footprint (none) -> Resistor_THT:R_Axial_DIN0309_L9.0mm_D3.2mm_P12.70mm_Horizontal; CatNo (none) -> CF12JT1M00TR-ND
- R10, R20, R22, R8: value 10k -> 10k 1/2W; footprint (none) -> Resistor_THT:R_Axial_DIN0309_L9.0mm_D3.2mm_P12.70mm_Horizontal; CatNo (none) -> S10KHTR-ND
- R11, R12, R15, R16, R5, R6: value 10k 3W -> 10k 5W; footprint (none) -> Resistor_THT:R_Axial_DIN0617_L17.0mm_D6.0mm_P25.40mm_Horizontal; CatNo (none) -> A142824CT-ND
- R13, R14: footprint (none) -> Resistor_THT:R_Axial_DIN0309_L9.0mm_D3.2mm_P12.70mm_Horizontal; CatNo (none) -> S1.8KHTR-ND
- R17, R18: value 120k 1W -> 120k 2W; footprint (none) -> Resistor_THT:R_Axial_DIN0309_L9.0mm_D3.2mm_P12.70mm_Horizontal; CatNo (none) -> 120KZTR-ND
- R3, R4: value 220 -> 220 1/2W; footprint (none) -> Resistor_THT:R_Axial_DIN0309_L9.0mm_D3.2mm_P12.70mm_Horizontal; CatNo (none) -> S220HTR-ND
- RV1, RV2: footprint (none) -> Vishay_Pot_148:Potentiometer_Vishay_148-149_Single_Horizontal; CatNo (none) -> 693-14910F0GJSX10253KA-ND
- U1, U2, U3: footprint Valve:Valve_Noval_P -> Octal_Sockets:AES-P-ST8-193; CatNo (none) -> AES P-ST8-193
Connections:
- net B+: now also C1.1
- net GND: now also C1.2, H1.1, H2.1, H3.1, H4.1, J3.3 (Pin_3)
- net at C9.1, R19.1: now also U2.4 (G); no longer U2.1 (G)
- net at J4.3 (Pin_3), R15.2: now also U2.5 (P); no longer U2.2 (A)
- net at U1.7 (F1), U2.7 (F1), U3.7 (F1): now also J3.1 (Pin_1)
- net at U1.8 (F2), U2.8 (F2), U3.8 (F2): now also J3.2 (Pin_2)
- net at C5.2, C7.1, R7.2: now also U2.1 (G); no longer U2.7 (4)
- net at C6.1, R6.2: now also U1.5 (P); no longer U1.2 (A)
- net at C6.2, C8.1, R9.2: now also U3.1 (G); no longer U3.7 (4)
- net at J4.2 (Pin_2), R11.2: now also U2.2 (P); no longer U2.5 (A)
- net at J4.4 (Pin_4), R12.2: now also U3.2 (P); no longer U3.5 (A)
- net at J4.5 (Pin_5), R16.2: now also U3.5 (P); no longer U3.2 (A)
- net at R1.2: now also J2.1 (Pin_1), U1.1 (G); no longer U1.7 (4)
- net at R2.2: now also J2.3 (Pin_3), U1.4 (G); no longer U1.1 (G)
- net at C3.1, R3.1: now also U1.3 (C); no longer U1.8 (6)
- net at C4.1, R4.1: now also U1.6 (C); no longer U1.3 (K)
- net at C5.1, R5.2: now also U1.2 (P); no longer U1.5 (A)
- net at C10.1, R21.1: now also U3.4 (G); no longer U3.1 (G)
- new net: R13.1, U2.3 (C), U2.6 (C)
- new net: R14.1, U3.3 (C), U3.6 (C)

Commit message: bom
Parts:
- J1: CatNo (none) -> WM2122-ND
- J3: CatNo (none) -> WM50010-03-ND
Changed lines of the file:
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@@
       (effects (font (size 1.27 1.27)) hide)
     )
+    (property "CatNo" "WM2122-ND" (id 4) (at 53.975 24.13 0))
     (pin "1")
     (pin "2")
@@
   )
   (symbol (lib_id "Connector_Generic:Conn_01x03") (at 57.15 187.96 0) (mirror y) (unit 1)
-    (in_bom yes) (on_board yes) (fields_autoplaced)
+    (in_bom yes) (on_board yes)
     (property "Reference" "J3" (id 0) (at 57.15 179.07 0))
     (property "Value" "Conn_01x03" (id 1) (at 57.15 181.61 0))
@@
       (effects (font (size 1.27 1.27)) hide)
     )
-    (pin "1")
-    (pin "2")
+    (property "CatNo" "WM50010-03-ND" (id 4) (at 53.975 194.31 0))
+    (pin "1")
+    (pin "2")
