File: hardware/dac/dac.kicad_pcb (KiCad board)
At the start: 2 copper layers, 116.8 x 111.8 mm, 55 parts, among them IC1 EC1110120201_with_knurled_SHA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, J1 Conn_01x04, J2 Conn_02x08_Odd_Even, J3 Conn_02x08_Odd_Even, J4 Conn_02x08_Odd_Even, J5 Conn_01x02, J6 Conn_01x04, J7 Conn_01x04, Q1 Q_PNP_BCE, SW1 SW_SPST, SW2 SW_SPST, U1 74HC4040, U2 74LS08, U3 74LS174, U4 74HCT245, U5 74LS138, U6 DS1306, U7 IM6402, U8 MAX503, U9 MAX503, X1 4.9152MHz, Y1 32.768 kHz

Commit message: PCB Rev 1 ready to fab?
Other:
- board text added: "+"
- board text added: "+5"
- board text added: "-"
- board text added: "-5"
- board text added: "1"
- board text added: "1200"
- board text added: "19.2k"
- board text added: "2400"
- board text added: "300"
- board text added: "38.4k"
- board text added: "4800"
- board text added: "600"
- board text added: "9600"
- board text added: "Batt 3V"
- board text added: "Baud Rate"
- board text added: "FT232 USB Serial"
- board text added: "G"
- board text added: "Scope Clock Display Rev 1 - Jan 2023 UPCO Graphics Systems"
- board text added: "XY Out"
- board text added: "Z Out"
