File: hardware/psu/psu.kicad_sch (KiCad schematic)
At the start: 66 parts, among them J1 Conn_01x02, J10 Conn_01x04, J12 Conn_01x02, J13 Conn_01x03, J14 Conn_01x05, J15 Conn_01x02, J2 Conn_01x05, J3 Conn_01x02, J4 Conn_01x06, J5 Conn_01x03, J6 Conn_01x05, J7 Conn_01x08, J8 Conn_01x03, J9 Conn_01x04, K1 PR16-12V-540-2C, Q1 Q_NMOS_GDS, SW1 SW_SPST, T1 AS-1T175, U1 LM7905_TO220, U2 BOM_item, U3 BOM_item

Commit message: PSU Rev A
Parts:
- added D12: LED, LED_THT:LED_D3.0mm, symbol Device:LED
- added R13: 3.3K, Resistor_THT:R_Axial_DIN0309_L9.0mm_D3.2mm_P12.70mm_Horizontal, symbol Device:R_US
- Q1: value Q_NMOS_GDS -> NMOS
- U2: value BOM_item -> BOM_item2; CatNo P-ST8-193 -> (25) WM2301-ND; Vendor AES -> DigiKey
- U3: value BOM_item -> BOM_item1
Connections:
- net +12V: now also R13.1
- net at K1.1, Q1.2 (D): now also D12.1 (K)
- new net: D12.2 (A), R13.2
Other:
- note added: "Crimp pin"
- note removed: "Octal Socket"
Changed lines of the file:
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@@
   (junction (at 215.9 96.52) (diameter 0) (color 0 0 0 0)
+  )
+  (junction (at 124.46 21.59) (diameter 0) (color 0 0 0 0)
   )
   (junction (at 223.52 58.42) (diameter 0) (color 0 0 0 0)
@@
     (stroke (width 0) (type default) (color 0 0 0 0))
   )
+  (wire (pts (xy 114.3 25.4) (xy 114.3 21.59))
+    (stroke (width 0) (type default) (color 0 0 0 0))
+  )
   (wire (pts (xy 223.52 44.45) (xy 223.52 48.26))
     (stroke (width 0) (type default) (color 0 0 0 0))
@@
     (stroke (width 0) (type default) (color 0 0 0 0))
   )
+  (wire (pts (xy 121.92 21.59) (xy 124.46 21.59))
+    (stroke (width 0) (type default) (color 0 0 0 0))
+  )
   (wire (pts (xy 229.87 116.84) (xy 229.87 125.73))
     (stroke (width 0) (type default) (color 0 0 0 0))
@@
     (stroke (width 0) (type default) (color 0 0 0 0))
   )
+  (wire (pts (xy 110.49 25.4) (xy 114.3 25.4))
+    (stroke (width 0) (type default) (color 0 0 0 0))
+  )
   (wire (pts (xy 137.16 87.63) (xy 137.16 90.17))
     (stroke (width 0) (type default) (color 0 0 0 0))
@@
     (stroke (width 0) (type default) (color 0 0 0 0))
   )
-  (wire (pts (xy 124.46 40.64) (xy 124.46 16.51))
+  (wire (pts (xy 124.46 40.64) (xy 124.46 21.59))
     (stroke (width 0) (type default) (color 0 0 0 0))
   )
@@
     (stroke (width 0) (type default) (color 0 0 0 0))
   )
+  (wire (pts (xy 124.46 21.59) (xy 124.46 16.51))
+    (stroke (width 0) (type default) (color 0 0 0 0))
+  )
   (wire (pts (xy 60.96 173.99) (xy 69.85 173.99))
     (stroke (width 0) (type default) (color 0 0 0 0))
@@
     (stroke (width 0) (type default) (color 0 0 0 0))
   )
+  (wire (pts (xy 97.79 25.4) (xy 102.87 25.4))
+    (stroke (width 0) (type default) (color 0 0 0 0))
+  )
   (wire (pts (xy 152.4 73.66) (xy 154.94 73.66))
     (stroke (width 0) (type default) (color 0 0 0 0))
@@
     (stroke (width 0) (type default) (color 0 0 0 0))
   )
-  (text "Octal Socket" (at 80.01 21.59 0)
+  (text "Crimp pin" (at 76.2 24.13 0)
     (effects (font (size 1.27 1.27)) (justify left bottom))
   )
@@
     (effects (font (size 1.905 1.905)) (justify left bottom))
   )
-  (text "5mm 24 pin breakaway header" (at 80.01 26.67 0)
+  (text "5mm 24 pin breakaway header" (at 76.2 19.05 0)
     (effects (font (size 1.27 1.27)) (justify left bottom))
   )
@@
     (pin "1")
   )
+  (symbol (lib_id "Device:LED") (at 118.11 21.59 180) (unit 1)
+    (in_bom yes) (on_board yes) (fields_autoplaced)
+    (property "Reference" "D12" (id 0) (at 119.6975 13.97 0))
+    (property "Value" "LED" (id 1) (at 119.6975 16.51 0))
+    (property "Footprint" "LED_THT:LED_D3.0mm" (id 2) (at 118.11 21.59 0)
+      (effects (font (size 1.27 1.27)) hide)
+    )
+    (property "Datasheet" "~" (id 3) (at 118.11 21.59 0)
+      (effects (font (size 1.27 1.27)) hide)
+    )
+    (pin "1")
+    (pin "2")
+  )
   (symbol (lib_id "Connector_Generic:Conn_01x04") (at 274.32 120.65 0) (unit 1)
     (in_bom yes) (on_board yes) (fields_autoplaced)
@@
     (pin "2")
   )
-  (symbol (lib_id "misc_bom:BOM_item") (at 49.53 26.67 0) (unit 1)
+  (symbol (lib_id "misc_bom:BOM_item") (at 45.72 19.05 0) (unit 1)
     (in_bom yes) (on_board no)
-    (property "Reference" "U3" (id 0) (at 58.42 22.86 0)
-      (effects (font (size 1.27 1.27)) hide)
-    )
-    (property "Value" "BOM_item" (id 1) (at 50.8 22.86 0)
-      (effects (font (size 1.27 1.27)) hide)
-    )
-    (property "Footprint" "" (id 2) (at 49.53 26.67 0)
-      (effects (font (size 1.27 1.27)) hide)
-    )
-    (property "Datasheet" "" (id 3) (at 49.53 26.67 0)
-      (effects (font (size 1.27 1.27)) hide)
-    )
-    (property "CatNo" "WM50000-24-ND" (id 4) (at 68.58 25.4 0))
-    (property "Vendor" "DigiKey" (id 5) (at 54.61 25.4 0))
+    (property "Reference" "U3" (id 0) (at 54.61 15.24 0)
+      (effects (font (size 1.27 1.27)) hide)
+    )
+    (property "Value" "BOM_item1" (id 1) (at 46.99 15.24 0)
+      (effects (font (size 1.27 1.27)) hide)
+    )
+    (property "Footprint" "" (id 2) (at 45.72 19.05 0)
+      (effects (font (size 1.27 1.27)) hide)
+    )
+    (property "Datasheet" "" (id 3) (at 45.72 19.05 0)
+      (effects (font (size 1.27 1.27)) hide)
+    )
+    (property "CatNo" "WM50000-24-ND" (id 4) (at 64.77 17.78 0))
+    (property "Vendor" "DigiKey" (id 5) (at 50.8 17.78 0))
   )
   (symbol (lib_id "power:GND") (at 113.03 81.28 0) (unit 1)
@@
     (pin "2")
   )
+  (symbol (lib_id "power:+12V") (at 97.79 25.4 0) (unit 1)
+    (in_bom yes) (on_board yes)
+    (property "Reference" "#PWR011" (id 0) (at 97.79 29.21 0)
+      (effects (font (size 1.27 1.27)) hide)
+    )
+    (property "Value" "+12V" (id 1) (at 93.98 25.4 0))
+    (property "Footprint" "" (id 2) (at 97.79 25.4 0)
+      (effects (font (size 1.27 1.27)) hide)
+    )
+    (property "Datasheet" "" (id 3) (at 97.79 25.4 0)
+      (effects (font (size 1.27 1.27)) hide)
+    )
+    (pin "1")
+  )
   (symbol (lib_id "Mechanical:MountingHole") (at 15.24 26.67 0) (unit 1)
     (in_bom yes) (on_board yes) (fields_autoplaced)
@@
     )
     (property "Datasheet" "~" (id 3) (at 74.93 176.53 0)
+      (effects (font (size 1.27 1.27)) hide)
+    )
+    (property "CatNo" "" (id 4) (at 74.93 176.53 0)
       (effects (font (size 1.27 1.27)) hide)
     )
@@
     (pin "2")
   )
-  (symbol (lib_id "misc_bom:BOM_item") (at 49.53 21.59 0) (unit 1)
-    (in_bom yes) (on_board no)
-    (property "Reference" "U2" (id 0) (at 58.42 17.78 0)
-      (effects (font (size 1.27 1.27)) hide)
-    )
-    (property "Value" "BOM_item" (id 1) (at 50.8 17.78 0)
-      (effects (font (size 1.27 1.27)) hide)
-    )
-    (property "Footprint" "" (id 2) (at 49.53 21.59 0)
-      (effects (font (size 1.27 1.27)) hide)
-    )
-    (property "Datasheet" "" (id 3) (at 49.53 21.59 0)
-      (effects (font (size 1.27 1.27)) hide)
-    )
-    (property "CatNo" "P-ST8-193" (id 4) (at 66.04 20.32 0))
-    (property "Vendor" "AES" (id 5) (at 54.61 20.32 0))
-  )
   (symbol (lib_id "Device:C_Polarized_Small_US") (at 208.28 88.9 0) (unit 1)
     (in_bom yes) (on_board yes)
@@
       (effects (font (size 1.27 1.27)) (justify left))
     )
-    (property "Value" "Q_NMOS_GDS" (id 1) (at 130.81 25.3999 0)
+    (property "Value" "NMOS" (id 1) (at 130.81 25.3999 0)
       (effects (font (size 1.27 1.27)) (justify left))
     )
@@
     (pin "2")
   )
+  (symbol (lib_id "misc_bom:BOM_item") (at 45.72 24.13 0) (unit 1)
+    (in_bom yes) (on_board no)
+    (property "Reference" "U2" (id 0) (at 54.61 20.32 0)
+      (effects (font (size 1.27 1.27)) hide)
+    )
+    (property "Value" "BOM_item2" (id 1) (at 46.99 20.32 0)
+      (effects (font (size 1.27 1.27)) hide)
+    )
+    (property "Footprint" "" (id 2) (at 45.72 24.13 0)
+      (effects (font (size 1.27 1.27)) hide)
+    )
+    (property "Datasheet" "" (id 3) (at 45.72 24.13 0)
+      (effects (font (size 1.27 1.27)) hide)
+    )
+    (property "CatNo" "(25) WM2301-ND" (id 4) (at 64.77 22.86 0))
+    (property "Vendor" "DigiKey" (id 5) (at 50.8 22.86 0))
+  )
   (symbol (lib_id "Device:C_Polarized_Small_US") (at 229.87 114.3 0) (unit 1)
     (in_bom yes) (on_board yes)
@@
     (pin "2")
   )
+  (symbol (lib_id "Device:R_US") (at 106.68 25.4 90) (unit 1)
+    (in_bom yes) (on_board yes)
+    (property "Reference" "R13" (id 0) (at 102.87 22.86 90))
+    (property "Value" "3.3K" (id 1) (at 109.22 22.86 90))
+    (property "Footprint" "Resistor_THT:R_Axial_DIN0309_L9.0mm_D3.2mm_P12.70mm_Horizontal" (id 2) (at 106.934 24.384 90)
+      (effects (font (size 1.27 1.27)) hide)
+    )
+    (property "Datasheet" "~" (id 3) (at 106.68 25.4 0)
+      (effects (font (size 1.27 1.27)) hide)
+    )
+    (pin "1")
+    (pin "2")
+  )
   (symbol (lib_id "Diode:1N4007") (at 166.37 82.55 270) (unit 1)
     (in_bom yes) (on_board yes)
@@
       (reference "#PWR010") (unit 1) (value "+12V") (footprint "")
     )
+    (path "/44bb1a09-bccd-496c-84af-2bf88fda89bc"
+      (reference "#PWR011") (unit 1) (value "+12V") (footprint "")
+    )
     (path "/2cc3a77d-b341-4bd3-a8a4-b85c466f20f7"
       (reference "#PWR012") (unit 1) (value "GND") (footprint "")
@@
       (reference "D11") (unit 1) (value "D_Bridge_+-AA") (footprint "Diode_THT:Diode_Bridge_19.0x3.5x10.0mm_P5.0mm")
     )
+    (path "/0b587c16-64d7-4f07-8130-e0161bf12ba2"
+      (reference "D12") (unit 1) (value "LED") (footprint "LED_THT:LED_D3.0mm")
+    )
     (path "/6cf244d9-2cf7-4f13-b2df-d892417e0130"
       (reference "D14") (unit 1) (value "D_Bridge_+-AA") (footprint "Diode_THT:Diode_Bridge_19.0x3.5x10.0mm_P5.0mm")
@@
     )
     (path "/bbee6bfb-df07-4535-8581-3336e8a8e5d4"
-      (reference "Q1") (unit 1) (value "Q_NMOS_GDS") (footprint "Package_TO_SOT_THT:TO-220-3_Vertical")
+      (reference "Q1") (unit 1) (value "NMOS") (footprint "Package_TO_SOT_THT:TO-220-3_Vertical")
     )
     (path "/2f8158ac-89f2-41e4-8db9-d3c0d43a940f"
@@
       (reference "R12") (unit 1) (value "10k") (footprint "Resistor_THT:R_Axial_DIN0309_L9.0mm_D3.2mm_P12.70mm_Horizontal")
     )
+    (path "/f020a3aa-ebaa-4dfe-bcda-0a1cb8e2dd80"
+      (reference "R13") (unit 1) (value "3.3K") (footprint "Resistor_THT:R_Axial_DIN0309_L9.0mm_D3.2mm_P12.70mm_Horizontal")
+    )
     (path "/c36e2220-14ee-481f-af40-a9fb4a4f5882"
       (reference "SW1") (unit 1) (value "SW_SPST") (footprint "Switch_8GA:8GA1016-Z")
@@
       (reference "U1") (unit 1) (value "LM7905_TO220") (footprint "Package_TO_SOT_THT:TO-220-3_Vertical")
     )
-    (path "/a11ebc0b-0f2f-4378-b51a-d55388d7654a"
-      (reference "U2") (unit 1) (value "BOM_item") (footprint "")
+    (path "/c66f0c80-ae79-4575-9459-59d70ffdc0c4"
+      (reference "U2") (unit 1) (value "BOM_item2") (footprint "")
     )
     (path "/1a98b841-a7d0-46b2-86ee-22bbe87fdffc"
-      (reference "U3") (unit 1) (value "BOM_item") (footprint "")
-    )
-  )
+      (reference "U3") (unit 1) (value "BOM_item1") (footprint "")
+    )
+  )
