File: hardware/psu/psu.kicad_pcb (KiCad board)
At the start: 2 copper layers, 177.8 x 114.3 mm, 66 parts, among them J1 Conn_01x02, J10 Conn_01x04, J11 Conn_01x03, J12 Conn_01x02, J13 Conn_01x03, J14 Conn_01x05, J15 Conn_01x02, J2 Conn_01x05, J3 Conn_01x02, J4 Conn_01x06, J5 Conn_01x03, J6 Conn_01x05, J7 Conn_01x08, J8 Conn_01x03, J9 Conn_01x04, K1 PR16-12V-540-2C, Q1 Q_NMOS_GDS, SW1 SW_SPST, U1 LM7905_TO220

Commit message: PSU layout done?
Parts:
- removed C16: 47u 400V, Capacitor_THT:CP_Radial_D12.5mm_P5.00mm
- removed D12: D_Bridge_+-AA, Diode_THT:Diode_Bridge_19.0x3.5x10.0mm_P5.0mm
- removed J11: Conn_01x03, Connector_Molex:Molex_KK-396_A-41791-0003_1x03_P3.96mm_Vertical
- removed JP1: WIRE_JUMPER, Connector_PinHeader_2.54mm:PinHeader_1x02_P2.54mm_Vertical
- added G***: LOGO, hv_danger:hv_danger, F.Cu at (161.9, 130.8)
- added R12: 10k, Resistor_THT:R_Axial_DIN0309_L9.0mm_D3.2mm_P12.70mm_Horizontal, F.Cu at (190.5, 101.6)
- moved J1 108.7 mm to (174.0, 29.2), turned to 90 degrees
- moved J6 108.2 mm to (97.8, 134.6), turned to 0 degrees
- moved J3 102.3 mm to (84.4, 29.3), turned to 0 degrees
- moved J15 88.5 mm to (199.4, 102.2)
- moved R9 85.1 mm to (127.0, 77.5), turned to 180 degrees
- moved Q1 70.6 mm to (199.1, 88.9), turned to 90 degrees
- moved J9 66.4 mm to (61.6, 117.5)
- moved R8 66.4 mm to (146.1, 77.5), turned to 180 degrees
- moved R11 58.6 mm to (189.2, 43.2), turned to 180 degrees
- moved J12 55.9 mm to (185.4, 29.2), turned to 90 degrees
- moved R7 45.8 mm to (166.4, 77.5), turned to 180 degrees
- moved C12 40.7 mm to (59.7, 77.5), turned to -90 degrees
- moved R10 36.5 mm to (189.2, 38.1), turned to 180 degrees
- moved J4 34.6 mm to (148.3, 133.9)
- moved R6 34.2 mm to (182.9, 106.7), turned to 90 degrees
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Connections:
- C14 pad 2: /0V -> GND
- C15 pad 2: /0V -> GND
- C3 pad 1: /0V -> GND
- C4 pad 2: /0V -> GND
- D1 pad 1: /0V -> GND
- D2 pad 2: /0V -> GND
- J10 pad 1: Net-(D14-Pad2) -> Net-(D11-Pad3)
- J10 pad 2: Net-(D14-Pad3) -> Net-(D11-Pad2)
- J10 pad 3: Net-(D11-Pad2) -> Net-(D14-Pad3)
- J10 pad 4: Net-(D11-Pad3) -> Net-(D14-Pad2)
- J3 pad 2: /0V -> GND
- J4 pad 3: /0V -> GND
- J6 pad 3: /115_A -> unconnected-(J6-Pad3)
- J6 pad 4: /115_B -> unconnected-(J6-Pad4)
- J7 pad 2: /0V -> GND
- J7 pad 4: /0V -> GND
- J7 pad 6: /6.3_1A -> /6.3_1B
- J9 pad 3: GND -> -5V
- R10 pad 1: /0V -> GND
- R11 pad 1: /0V -> GND
- R7 pad 1: /0V -> GND
Routing:
- net /SW_ACL: track 0.00 -> 179.8 mm
- net /ACN: track 0.00 -> 160.7 mm
- net /+360: track 0.00 -> 158.1 mm
- net +12V: track 0.00 -> 149.9 mm, vias 0 -> 1
- net /S4: track 0.00 -> 94.1 mm, vias 0 -> 1
- net /175_1A: track 0.00 -> 64.6 mm
- net GND: track 0.00 -> 62.3 mm
- net Net-(F1-Pad1): track 0.00 -> 56.1 mm
- net Net-(C1-Pad2): track 0.00 -> 54.8 mm
- net Net-(D14-Pad2): track 0.00 -> 53.3 mm
- net /S6: track 0.00 -> 51.4 mm, vias 0 -> 1
- net /S5: track 0.00 -> 48.2 mm
- net /-V_CRT: track 0.00 -> 46.9 mm
- net -5V: track 0.00 -> 46.0 mm
- net Net-(C2-Pad2): track 0.00 -> 44.1 mm
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- added copper zone on B.Cu, net GND
Other:
- board text added: "++"
- board text added: "+12"
- board text added: "+360"
- board text added: "-"
- board text added: "-1200"
- board text added: "-5"
- board text added: "CAUTION 1200V!"
- board text added: "CRT FIL"
- board text added: "CRT HV OUT"
- board text added: "CRT HV SECONDARY"
- board text added: "DC TO LOGIC"
- board text added: "DC XFRMR SECONDARIES"
- board text added: "DEFL AMP B+"
- board text added: "DEFL PRIMARY"
- board text added: "HV ENA"
- board text added: "HV PRIMARY"
- board text added: "LV PRIMARY"
- board text added: "SPARE FIL"
- board text added: "UPCO Scope Clock Power Supply Rev A - 2023-02"
- board text added: "~"

Commit message: PSU Rev A
Parts:
- added D12: LED, LED_THT:LED_D3.0mm, F.Cu at (191.8, 110.5)
- added R13: 3.3K, Resistor_THT:R_Axial_DIN0309_L9.0mm_D3.2mm_P12.70mm_Horizontal, F.Cu at (188.0, 88.9)
- Q1: value Q_NMOS_GDS -> NMOS
- moved R12 1.91 mm to (192.4, 101.6)
Routing:
- net Net-(K1-Pad1): track 21.1 -> 48.5 mm
- net +12V: track 149.9 -> 171.6 mm, vias 1 -> 2
- net Net-(D12-Pad2): track 0.00 -> 9.42 mm
- net Net-(J15-Pad1): track 22.0 -> 20.1 mm
Other:
- board text added: "HV ON"
