File: hardware/dac_mods/dac_mods.kicad_sch (KiCad schematic)
At the start: 2 parts

Commit message: software tweaks, working on case
Connections:
- net DAC_X_WR: now also U?.12 (O0); no longer U?.4 (O0)
- net DAC_Y_WR: now also U?.11 (O1); no longer U?.5 (O1)
- net GND: now also U?.14 (A0); no longer U?.2 (A0)
- net nDACX: now also U?.15 (E); no longer U?.1 (E)
- net at U?.13 (Q1): now also U?.13 (A1); no longer U?.3 (A1)
Changed lines of the file:
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@@
     (pin "9")
   )
-  (symbol (lib_id "74xx:74LS139") (at 154.94 64.77 0) (unit 1)
+  (symbol (lib_id "74xx:74LS139") (at 154.94 64.77 0) (unit 2)
     (in_bom yes) (on_board yes) (fields_autoplaced)
     (property "Reference" "U?" (id 0) (at 154.94 54.61 0))
@@
     )
     (path "/f76bfdec-a6b1-47b5-998c-b7d469cbdb07"
-      (reference "U?") (unit 1) (value "74LS139") (footprint "")
+      (reference "U?") (unit 2) (value "74LS139") (footprint "")
     )
   )
