File: hardware/b_250_test/b_250_test.kicad_pcb (KiCad board)
At the start: 2 copper layers, 14 parts, among them J1 Conn_01x02, J2 Conn_01x03

Commit message: working on 6T9 version of sound
Parts:
- C1: footprint Connector_TE-Connectivity:TE_826576-2_1x02_P3.96mm_Vertical -> Capacitor_THT:CP_Radial_D22.0mm_P10.00mm_SnapIn
- moved J1 57.4 mm to (31.0, 53.3), turned to -90 degrees

Commit message: working on 6T9 design
Parts:
- added C11: 0.1uF, Capacitor_THT:C_Disc_D3.4mm_W2.1mm_P2.50mm, F.Cu at (149.0, 62.5)
- added C12: 0.1uF, Capacitor_THT:C_Disc_D3.4mm_W2.1mm_P2.50mm, F.Cu at (149.0, 66.2)
- added C13: 2.2uF, Capacitor_THT:C_Disc_D3.4mm_W2.1mm_P2.50mm, F.Cu at (149.0, 69.8)
- added H1: MountingHole, MountingHole:MountingHole_4.3mm_M4, F.Cu at (130.7, 62.1)
- added H2: MountingHole, MountingHole:MountingHole_4.3mm_M4, F.Cu at (130.7, 72.3)
- added H3: MountingHole, MountingHole:MountingHole_4.3mm_M4, F.Cu at (130.7, 82.5)
- added H4: MountingHole, MountingHole:MountingHole_4.3mm_M4, F.Cu at (130.7, 92.6)
- added J3: Conn_01x02, Connector_PinHeader_2.54mm:PinHeader_1x02_P2.54mm_Vertical, F.Cu at (160.0, 59.4)
- added J4: AVR-ISP-6, Connector_PinHeader_2.54mm:PinHeader_2x03_P2.54mm_Vertical, F.Cu at (149.7, 88.2)
- added J5: Conn_01x04, Connector_PinHeader_2.54mm:PinHeader_1x04_P2.54mm_Vertical, F.Cu at (164.0, 74.0)
- added JP1: JP2, Connector_PinHeader_2.54mm:PinHeader_1x02_P2.54mm_Vertical, F.Cu at (164.7, 59.4)
- added R14: 10k, Resistor_THT:R_Axial_DIN0204_L3.6mm_D1.6mm_P5.08mm_Horizontal, F.Cu at (154.5, 69.0)
- added RV1: 100k_audio, Potentiometer_THT:Potentiometer_Bourns_3266Y_Vertical, F.Cu at (161.3, 88.9)
- added T1: AES_PT-31, my_trans:AES-PT-31, F.Cu at (134.0, 135.9)
- added U2: SN76489, Package_DIP:DIP-16_W7.62mm_LongPads, F.Cu at (137.8, 59.1)
- added U3: ATtiny84A-P, Package_DIP:DIP-14_W7.62mm, F.Cu at (137.4, 81.0)
- added X1: CXO_DIP8, Oscillator:Oscillator_DIP-8, F.Cu at (150.7, 82.6)
- C5: value 10uF 400V -> 0.1uF; footprint Capacitor_THT:CP_Radial_D10.0mm_P5.00mm -> Capacitor_THT:C_Disc_D3.4mm_W2.1mm_P2.50mm
- J2: value Conn_01x03 -> Conn_01x02; footprint Connector_TE-Connectivity:TE_826576-3_1x03_P3.96mm_Vertical -> Connector_PinHeader_2.54mm:PinHeader_1x02_P2.54mm_Vertical
- R5: value 47k 2W -> 1; footprint Resistor_THT:R_Axial_DIN0414_L11.9mm_D4.5mm_P20.32mm_Horizontal -> Resistor_THT:R_Axial_DIN0204_L3.6mm_D1.6mm_P5.08mm_Horizontal
- moved C5 77.4 mm to (149.0, 58.9)
- moved R5 74.3 mm to (154.5, 65.8)
- moved J2 72.6 mm to (155.4, 59.4)
Connections:
- net Net-(C1-Pad2) renamed /HTX
- C5 pad 1: Net-(J2-Pin_2) -> GND
- C5 pad 2: Earth -> +5V
- J2 pad 1: HT -> Net-(J2-Pin_1)
- J2 pad 2: Net-(J2-Pin_2) -> GND
- R5 pad 1: HT -> GND
- R5 pad 2: Net-(J2-Pin_2) -> Earth

Commit message: working on placement
Parts:
- added C10: 0.22uF 400V, Capacitor_THT:C_Rect_L16.5mm_W6.0mm_P15.00mm_MKT, F.Cu at (-43.6, 101.5)
- added C6: 100uF 16V, Capacitor_THT:CP_Radial_D5.0mm_P2.00mm, F.Cu at (162.6, 132.1)
- added C7: 10uF 450V, Capacitor_THT:CP_Radial_D10.0mm_P5.00mm, F.Cu at (128.3, 99.2)
- added C8: 0.22uF 400V, Capacitor_THT:C_Rect_L16.5mm_W6.0mm_P15.00mm_MKT, F.Cu at (-43.6, 93.9)
- added C9: 330pF 100V, Capacitor_THT:C_Rect_L7.2mm_W4.5mm_P5.00mm_FKS2_FKP2_MKS2_MKP2, F.Cu at (-15.5, 97.9)
- added J6: Conn_01x02, Connector_TE-Connectivity:TE_826576-2_1x02_P3.96mm_Vertical, F.Cu at (-24.1, 99.1)
- added LS1: Speaker, Connector_TE-Connectivity:TE_826576-2_1x02_P3.96mm_Vertical, F.Cu at (183.4, 30.0)
- added R10: 47k, Resistor_THT:R_Axial_DIN0309_L9.0mm_D3.2mm_P12.70mm_Horizontal, F.Cu at (170.2, 94.0)
- added R11: 470K, Resistor_THT:R_Axial_DIN0207_L6.3mm_D2.5mm_P10.16mm_Horizontal, F.Cu at (138.4, 133.3)
- added R12: 33K, Resistor_THT:R_Axial_DIN0207_L6.3mm_D2.5mm_P10.16mm_Horizontal, F.Cu at (-43.9, 119.4)
- added R13: 270k, Resistor_THT:R_Axial_DIN0207_L6.3mm_D2.5mm_P10.16mm_Horizontal, F.Cu at (138.4, 124.5)
- added R15: 330, Resistor_THT:R_Axial_DIN0204_L3.6mm_D1.6mm_P7.62mm_Horizontal, F.Cu at (-18.9, 118.0)
- added R6: 1K, Resistor_THT:R_Axial_DIN0207_L6.3mm_D2.5mm_P10.16mm_Horizontal, F.Cu at (-43.9, 107.3)
- added R7: 270 1W, Resistor_THT:R_Axial_DIN0411_L9.9mm_D3.6mm_P15.24mm_Horizontal, F.Cu at (154.9, 137.2)
- added R8: 2.2K, Resistor_THT:R_Axial_DIN0207_L6.3mm_D2.5mm_P10.16mm_Horizontal, F.Cu at (138.4, 128.3)
- added R9: 120K, Resistor_THT:R_Axial_DIN0414_L11.9mm_D4.5mm_P15.24mm_Horizontal, F.Cu at (138.4, 109.2)
- added SW1: SW_SPST, Connector_PinHeader_2.54mm:PinHeader_1x02_P2.54mm_Vertical, F.Cu at (-11.4, 121.9)
- added U1: 6T9, my_tubes:Compactron_PCB, F.Cu at (161.3, 113.0)
- C1: footprint Capacitor_THT:CP_Radial_D22.0mm_P10.00mm_SnapIn -> my_tubes:Compactron_PCB
- R5: footprint Resistor_THT:R_Axial_DIN0204_L3.6mm_D1.6mm_P5.08mm_Horizontal -> Resistor_THT:R_Axial_DIN0309_L9.0mm_D3.2mm_P12.70mm_Horizontal
- T1: footprint my_trans:AES-PT-31 -> my_trans:MPS-OT8SE
- moved C11 182.7 mm to (-32.6, 42.2)
- moved C12 182.7 mm to (-32.6, 45.9)
- moved C13 182.7 mm to (-32.6, 49.5)
- moved C5 182.7 mm to (-32.6, 38.6)
- moved J4 182.7 mm to (-31.9, 67.9)
- moved J5 182.7 mm to (-17.6, 53.7)
- moved JP1 182.7 mm to (-16.9, 39.1)
- moved U3 182.7 mm to (-44.2, 60.7)
- moved J2 182.7 mm to (-26.2, 39.1)
- moved J3 182.7 mm to (-21.6, 39.1)
- moved R14 182.7 mm to (-27.1, 48.7)
- moved R5 182.7 mm to (-27.1, 45.5)
- moved RV1 182.7 mm to (-20.3, 68.6)
- moved U2 182.7 mm to (-43.8, 38.8)
- moved X1 182.7 mm to (-30.9, 62.3)
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Connections:
- U2 pad 6: unconnected-(U2-nCE-Pad6) -> GND
Other:
- board outline added: 177.8 x 114.3 mm

Commit message: first pass place & route
Parts:
- C1: footprint my_tubes:Compactron_PCB -> Capacitor_THT:CP_Radial_D22.0mm_P10.00mm_SnapIn
- moved R6 226.7 mm to (182.2, 91.4), turned to 180 degrees
- moved R15 212.7 mm to (193.0, 99.8), turned to -90 degrees
- moved J6 210.0 mm to (185.9, 100.6), turned to -90 degrees
- moved SW1 193.7 mm to (182.1, 130.0), turned to 90 degrees
- moved C8 186.5 mm to (142.7, 88.0), turned to -90 degrees
- moved R12 185.9 mm to (141.6, 130.8)
- moved C9 162.0 mm to (141.6, 137.2)
- moved C10 154.7 mm to (110.4, 115.8)
- moved J4 149.1 mm to (111.8, 28.0)
- moved U2 148.7 mm to (104.1, 53.3), turned to -90 degrees
- moved C11 141.2 mm to (108.0, 55.9), turned to -90 degrees
- moved X1 137.1 mm to (105.4, 77.5), turned to 90 degrees
- moved R5 135.1 mm to (95.2, 102.9), turned to -90 degrees
- moved R14 133.4 mm to (105.4, 33.0), turned to 90 degrees
- moved J3 133.1 mm to (99.1, 95.2)
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Connections:
- net Net-(U1B-S) renamed /HT_G
- R15 pad 2: GND -> Earth
Routing:
- net HT: track 0.00 -> 179.4 mm
- net Net-(SW1-B): track 0.00 -> 136.1 mm
- net /HT_M2: track 0.00 -> 49.8 mm
- net Net-(U1B-G2): track 0.00 -> 48.3 mm
- net Net-(J2-Pin_1): track 0.00 -> 46.9 mm
- net /HT_M1: track 0.00 -> 44.9 mm
- net Net-(SW1-A): track 0.00 -> 44.3 mm
- net /SCL: track 0.00 -> 42.7 mm
- net /HT_M3: track 0.00 -> 38.5 mm
- net /MISO: track 0.00 -> 37.6 mm, vias 0 -> 1
- net Net-(J6-Pin_1): track 0.00 -> 35.3 mm
- net /HTP: track 0.00 -> 33.7 mm
- net /HTPRE: track 0.00 -> 33.5 mm
- net Net-(U1A-K1): track 0.00 -> 32.8 mm
- net /MOSI: track 0.00 -> 30.7 mm, vias 0 -> 1
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- added copper zone on F.Cu, net +5V
- added copper zone on B.Cu, net Earth
- added copper zone on B.Cu, net GND

Commit message: tweaking
Parts:
- moved C8 9.64 mm to (134.6, 93.2)
- moved R9 7.07 mm to (142.4, 102.1)
- moved C7 5.67 mm to (124.4, 93.2)
- moved C9 4.94 mm to (146.2, 135.3)
- moved R12 2.36 mm to (143.4, 129.3)
Routing:
- net Net-(SW1-A): track 44.3 -> 0.00 mm
- net Net-(U1A-K1): track 32.8 -> 8.55 mm
- net /HTP: track 33.7 -> 24.7 mm
- net Net-(U1B-G2): track 48.3 -> 50.2 mm
- net /HTPRE: track 33.5 -> 34.1 mm
