File: hardware/b_250_test/b_250_test.kicad_pcb (KiCad board)
At the start: 2 copper layers, 177.8 x 114.3 mm, 49 parts, among them J1 Conn_01x02, J2 Conn_01x02, J3 Conn_01x02, J4 AVR-ISP-6, J5 Conn_01x04, J6 Conn_01x02, SW1 SW_SPST, T1 AES_PT-31, U1 6T9, U2 SN76489, U3 ATtiny84A-P, X1 CXO_DIP8

Commit message: silkscreen and minor tweaks
Parts:
- moved R7 34.3 mm to (191.3, 126.4), turned to 180 degrees
- moved SW1 16.3 mm to (166.5, 134.6)
Routing:
- net Net-(U1A-K1): track 8.55 -> 32.6 mm
- net Net-(SW1-A): track 0.00 -> 22.0 mm
- net Net-(SW1-B): track 136.1 -> 150.7 mm
Other:
- board text added: "(TEST LOAD)"
- board text added: "+5 Rx Tx GND"
- board text added: "120VAC"
- board text added: "6.3VAC (fil)"
- board text added: "AMP in"
- board text added: "B+ 250V"
- board text added: "ISP"
- board text added: "NFB"
- board text added: "PSG out"
- board text added: "SPKR 8R"
- board text added: "UPCO Graphics Systems Sound Card V1.0 E. Hazen - 2024-03"
- board text added: "VOL"
