File: hardware/b_250_test/b_250_test.kicad_sch (KiCad schematic)
At the start: 15 parts, among them J1 Conn_01x02, J2 Conn_01x03

Commit message: working on 6T9 version of sound
Parts:
- removed C5: 10uF 400V, Capacitor_THT:CP_Radial_D10.0mm_P5.00mm, symbol Device:C
- removed J2: Conn_01x03, Connector_TE-Connectivity:TE_826576-3_1x03_P3.96mm_Vertical, symbol Connector_Generic:Conn_01x03
- removed R5: 47k 2W, Resistor_THT:R_Axial_DIN0414_L11.9mm_D4.5mm_P20.32mm_Horizontal, symbol Device:R_US
- added C10, C8: 0.22uF 400V, symbol Device:C
- added C6: 100uF 16V, symbol Device:C
- added C7: 10uF 450V, symbol Device:C
- added C9: 330pF 100V, symbol Device:C
- added LS1: Speaker, symbol Device:Speaker
- added R10: 1K, symbol Device:R_US
- added R11: 470K, symbol Device:R_US
- added R12: 33K, symbol Device:R_US
- added R13, R8: 2.2K, symbol Device:R_US
- added R7: 270 1W, symbol Device:R_US
- added R9: 120K, symbol Device:R_US
- added T1: AES_PT-31, symbol my_tubes:AES_PT-31
- added U1: ~, symbol my_tubes:6T9
- C1: footprint Connector_TE-Connectivity:TE_826576-2_1x02_P3.96mm_Vertical -> Capacitor_THT:CP_Radial_D22.0mm_P10.00mm_SnapIn
- R6: value 7k 15W -> 1K
Connections:
- net Earth: now also C6.2, C7.2, LS1.1, R11.1, R13.1, R7.1, R8.1, T1.3 (BLK), U1.6 (IS); no longer J1.2 (Pin_2), R6.2
- net HT: now also R6.2, R10.2, T1.1 (BLU); no longer R6.1
- net HT_IN: no longer J1.1 (Pin_1)
- new net: C6.1, R7.2, U1.9 (K2)
- new net: C7.1, R10.1, R9.2
- new net: C8.1, R9.1, U1.2 (P2)
- new net: C10.2, R13.2, U1.4 (G1)
- new net: C9.1, R12.1, R8.2, U1.5 (K1)
- new net: C9.2, LS1.2, R12.2, T1.4 (GRN)
- new net: C8.2, R11.2, U1.8 (G2)
- new net: R6.1, U1.10 (S)
- new net LOUT: T1.2 (RED), U1.11 (P2)
Other:
- note removed: "Test Load 36mA"
- moved on the sheet: C1, C2, C3, C4, D1, D2, J1, R1, R2, R3, R4

Commit message: working on 6T9 design
Parts:
- added C11, C12, C5: 0.1uF, Capacitor_THT:C_Disc_D3.4mm_W2.1mm_P2.50mm, symbol Device:C
- added C13: 2.2uF, Capacitor_THT:C_Disc_D3.4mm_W2.1mm_P2.50mm, symbol Device:C
- added H1, H2, H3, H4: MountingHole, MountingHole:MountingHole_4.3mm_M4, symbol Mechanical:MountingHole
- added J2, J3: Conn_01x02, Connector_PinHeader_2.54mm:PinHeader_1x02_P2.54mm_Vertical, symbol Connector_Generic:Conn_01x02
- added J4: AVR-ISP-6, Connector_PinHeader_2.54mm:PinHeader_2x03_P2.54mm_Vertical, symbol Connector:AVR-ISP-6
- added J5: Conn_01x04, Connector_PinHeader_2.54mm:PinHeader_1x04_P2.54mm_Vertical, symbol Connector_Generic:Conn_01x04
- added JP1: JP2, Connector_PinHeader_2.54mm:PinHeader_1x02_P2.54mm_Vertical, symbol Jumper:Jumper_2_Bridged
- added R14: 10k, Resistor_THT:R_Axial_DIN0204_L3.6mm_D1.6mm_P5.08mm_Horizontal, symbol Device:R_US
- added R5: 1, Resistor_THT:R_Axial_DIN0204_L3.6mm_D1.6mm_P5.08mm_Horizontal, symbol Device:R_US
- added RV1: 100k_audio, Potentiometer_THT:Potentiometer_Bourns_3266Y_Vertical, symbol amp-rescue:R_POT_US-Device
- added U2: SN76489, Package_DIP:DIP-16_W7.62mm_LongPads, symbol my_psg:SN76489
- added U3: ATtiny84A-P, Package_DIP:DIP-14_W7.62mm, symbol MCU_Microchip_ATtiny:ATtiny84A-P
- added X1: CXO_DIP8, Oscillator:Oscillator_DIP-8, symbol Oscillator:CXO_DIP8
- T1: footprint (none) -> my_trans:AES-PT-31
- U1: value ~ -> 6T9
Connections:
- net Earth: now also J1.2 (Pin_2), J3.2 (Pin_2), R5.2, RV1.1
- net HT_IN: now also J1.1 (Pin_1)
- net HTPRE: now reaches C7.1, R10.1, R9.2
- net HTP: now reaches C8.1, R9.1, U1.2 (P2)
- net HTX: now reaches C1.2, R1.2
- net at C10.1: now also RV1.2
- net LOUT renamed HT_OUT
- new net: C12.1, J2.1 (Pin_1), U2.7 (AOUT)
- new net: C12.2, JP1.1 (A)
- new net: U2.10 (D7), U3.13 (AREF/PA0)
- new net: U2.11 (D6), U3.12 (PA1)
- new net: U2.12 (D5), U3.11 (PA2)
- new net: U2.13 (D4), U3.10 (PA3)
- new net: U2.3 (D0), U3.6 (PA7)
- new net: U2.5 (nWE), U3.2 (XTAL1/PB0)
- new net: J3.1 (Pin_1), JP1.2 (B), RV1.3
- new net +5V: C11.2, C13.2, C5.2, J5.1 (Pin_1), U2.16 (VCC), U3.1 (VCC), X1.8 (Vcc)
- new net CLK: U2.14 (CLK), X1.5 (OUT)
- new net GND: C11.1, C13.1, C5.1, J2.2 (Pin_2), J4.6 (GND), J5.4 (Pin_4), R5.1, U2.8 (GND), U3.14 (GND), X1.4 (GND)
- new net MISO: J4.1 (MISO), U2.1 (D2), U3.8 (PA5)
- new net MOSI: J4.4 (MOSI), U2.2 (D1), U3.7 (PA6)
- new net RXD: J5.2 (Pin_2), U3.3 (XTAL2/PB1)
- new net SCL: J4.3 (SCK), U2.15 (D3), U3.9 (PA4)
- new net TXD: J5.3 (Pin_3), U3.5 (PB2)
- new net VCC: J4.2 (VCC), R14.2
- new net nRESET: J4.5 (~{RST}), R14.1, U3.4 (~{RESET}/PB3)
Other:
- note added: "PSG"
- moved on the sheet: C1, C10, C2, C3, C4, C6, C7, C8, C9, D1, D2, J1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

Commit message: working on placement
Parts:
- added J6: Conn_01x02, Connector_TE-Connectivity:TE_826576-2_1x02_P3.96mm_Vertical, symbol Connector_Generic:Conn_01x02
- added R15: 330, Resistor_THT:R_Axial_DIN0204_L3.6mm_D1.6mm_P7.62mm_Horizontal, symbol Device:R_US
- added SW1: SW_SPST, Connector_PinHeader_2.54mm:PinHeader_1x02_P2.54mm_Vertical, symbol Switch:SW_SPST
- C1: footprint Capacitor_THT:CP_Radial_D22.0mm_P10.00mm_SnapIn -> my_tubes:Compactron_PCB
- C10, C8: footprint (none) -> Capacitor_THT:C_Rect_L16.5mm_W6.0mm_P15.00mm_MKT; CatNo (none) -> 1572-1209-ND; MfgNo (none) -> 224MMR400K
- C13: CatNo (none) -> 445-181743-ND; MfgNo (none) -> FG18X5R1E225KRT00
- C6: footprint (none) -> Capacitor_THT:CP_Radial_D5.0mm_P2.00mm; symbol Device:C -> Device:C_Polarized; CatNo (none) -> 732-8598-1-ND; MfgNo (none) -> 860010372006
- C7: footprint (none) -> Capacitor_THT:CP_Radial_D10.0mm_P5.00mm; CatNo (none) -> 1189-1894-ND; MfgNo (none) -> 450BXC10MEFC10X20
- C9: footprint (none) -> Capacitor_THT:C_Rect_L7.2mm_W4.5mm_P5.00mm_FKS2_FKP2_MKS2_MKP2; CatNo (none) -> 1928-1236-ND; MfgNo (none) -> FKP2D003301D00JSSD
- D1, D2: CatNo (none) -> 4878-1N4007TR-ND; MfgNo (none) -> 1N4007
- LS1: footprint (none) -> Connector_TE-Connectivity:TE_826576-2_1x02_P3.96mm_Vertical
- R10: value 1K -> 47k; footprint (none) -> Resistor_THT:R_Axial_DIN0309_L9.0mm_D3.2mm_P12.70mm_Horizontal; CatNo (none) -> A142744CT-ND; MfgNo (none) -> ROX05SJ47K
- R11: footprint (none) -> Resistor_THT:R_Axial_DIN0207_L6.3mm_D2.5mm_P10.16mm_Horizontal; CatNo (none) -> BC4420CT-ND; MfgNo (none) -> VR25000004703JA500
- R12: footprint (none) -> Resistor_THT:R_Axial_DIN0207_L6.3mm_D2.5mm_P10.16mm_Horizontal; CatNo (none) -> CF14JT33K0TR-ND; MfgNo (none) -> CF14JT33K0
- R13: value 2.2K -> 270k; footprint (none) -> Resistor_THT:R_Axial_DIN0207_L6.3mm_D2.5mm_P10.16mm_Horizontal; CatNo (none) -> PPCQJ270KTR-ND; MfgNo (none) -> HVR2500002703JR500
- R5: footprint Resistor_THT:R_Axial_DIN0204_L3.6mm_D1.6mm_P5.08mm_Horizontal -> Resistor_THT:R_Axial_DIN0309_L9.0mm_D3.2mm_P12.70mm_Horizontal; CatNo (none) -> CF12JT1R00; MfgNo (none) -> CF12JT1R00
- R6: footprint (none) -> Resistor_THT:R_Axial_DIN0207_L6.3mm_D2.5mm_P10.16mm_Horizontal; CatNo (none) -> A142704CT-ND; MfgNo (none) -> ROX05SJ1K0
- R7: footprint (none) -> Resistor_THT:R_Axial_DIN0411_L9.9mm_D3.6mm_P15.24mm_Horizontal; CatNo (none) -> A131452CT-ND; MfgNo (none) -> ROX1SJ270R
- R8: footprint (none) -> Resistor_THT:R_Axial_DIN0207_L6.3mm_D2.5mm_P10.16mm_Horizontal; CatNo (none) -> A142712CT-ND; MfgNo (none) -> ROX05SJ2K2
- R9: footprint (none) -> Resistor_THT:R_Axial_DIN0414_L11.9mm_D4.5mm_P15.24mm_Horizontal; CatNo (none) -> 56-HVR3700001203JR500TR-ND; MfgNo (none) -> HVR3700001203JR500
- RV1: CatNo xxx -> 693-14910F0GJSX10104KA-ND
- T1: footprint my_trans:AES-PT-31 -> my_trans:MPS-OT8SE; symbol my_tubes:AES_PT-31 -> my_tubes:MPS-OT8SE
- U1: footprint (none) -> my_tubes:Compactron_PCB
Connections:
- net GND: now also U2.6 (nCE), R15.2
- net at LS1.2, T1.4 (YEL): now also SW1.2 (B); no longer C9.2, R12.2
- net at U1.1 (H1): now also J6.1 (Pin_1), R15.1
- net at U1.12 (H2): now also J6.2 (Pin_2)
- new net: C9.2, R12.2, SW1.1 (A)
Other:
- note added: "6.3V Heater"
- note added: "NFB"
- moved on the sheet: U1C

Commit message: first pass place & route
Parts:
- C1: footprint my_tubes:Compactron_PCB -> Capacitor_THT:CP_Radial_D22.0mm_P10.00mm_SnapIn
Connections:
- net Earth: now also R15.2
- net GND: no longer R15.2
- net HT_G: now reaches R6.1, U1.10 (S)
Changed lines of the file:
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@@
+    (effects (font (size 1.27 1.27)) (justify left bottom))
+  )
+  (label "HT_G" (at 219.075 108.585 90) (fields_autoplaced)
     (effects (font (size 1.27 1.27)) (justify left bottom))
   )
@@
         (path "/e2fa5dec-5d31-4df4-ad5f-66591cd37f62"
           (reference "C12") (unit 1)
+        )
+      )
+    )
+  )
+  (symbol (lib_id "power:Earth") (at 142.875 193.04 0) (unit 1)
+    (in_bom yes) (on_board yes) (dnp no)
+    (property "Reference" "#PWR026" (at 142.875 199.39 0)
+      (effects (font (size 1.27 1.27)) hide)
+    )
+    (property "Value" "Earth" (at 142.875 196.85 0)
+      (effects (font (size 1.27 1.27)) hide)
+    )
+    (property "Footprint" "" (at 142.875 193.04 0)
+      (effects (font (size 1.27 1.27)) hide)
+    )
+    (property "Datasheet" "~" (at 142.875 193.04 0)
+      (effects (font (size 1.27 1.27)) hide)
+    )
+    (pin "1")
+    (instances
+      (project "b_250_test"
+        (path "/e2fa5dec-5d31-4df4-ad5f-66591cd37f62"
+          (reference "#PWR026") (unit 1)
         )
       )
@@
       (effects (font (size 1.27 1.27)))
     )
-    (property "Footprint" "my_tubes:Compactron_PCB" (at 180.34 27.305 0)
+    (property "Footprint" "Capacitor_THT:CP_Radial_D22.0mm_P10.00mm_SnapIn" (at 180.34 27.305 0)
       (effects (font (size 1.27 1.27)) hide)
     )
@@
         )
       )
-    )
-  )
-  (symbol (lib_id "power:GND") (at 142.875 193.04 0) (unit 1)
-    (in_bom yes) (on_board yes) (dnp no)
-    (property "Reference" "#PWR026" (at 142.875 199.39 0)
-      (effects (font (size 1.27 1.27)) hide)
-    )
-    (property "Value" "GND" (at 146.05 193.04 0)
-      (effects (font (size 1.27 1.27)))
-    )
-    (property "Footprint" "" (at 142.875 193.04 0)
-      (effects (font (size 1.27 1.27)) hide)
-    )
-    (property "Datasheet" "" (at 142.875 193.04 0)
-      (effects (font (size 1.27 1.27)) hide)
-    )
-    (pin "1")
-    (instances
-      (project "b_250_test"
-        (path "/e2fa5dec-5d31-4df4-ad5f-66591cd37f62"
-          (reference "#PWR026") (unit 1)
-        )
-      )

Commit message: parts parts parts
Parts:
- C11, C12, C5: CatNo (none) -> 399-C321C104Z5U5TA-ND; MfgNo (none) -> C321C104Z5U5TA
- J1, J6, LS1: CatNo (none) -> WM50000-02-ND; MfgNo (none) -> 0416710001
- J4: CatNo 10129381-906002BLF-ND -> (none)
- U3: CatNo (none) -> ATTINY84A-PU-ND; MfgNo (none) -> ATTINY84A-PU
- X1: CatNo (none) -> XC235-ND; MfgNo (none) -> XC235-ND
Changed lines of the file:
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@@
+      (effects (font (size 1.27 1.27)) hide)
+    )
+    (property "CatNo" "399-C321C104Z5U5TA-ND" (at 109.22 99.695 0)
+      (effects (font (size 1.27 1.27)) hide)
+    )
+    (property "MfgNo" "C321C104Z5U5TA" (at 109.22 99.695 0)
       (effects (font (size 1.27 1.27)) hide)
     )
@@
       (effects (font (size 1.27 1.27)) hide)
     )
-    (property "CatNo" "10129381-906002BLF-ND" (at 108.585 154.94 0)
+    (property "CatNo" "" (at 108.585 154.94 0)
       (effects (font (size 1.27 1.27)))
     )
@@
       (effects (font (size 1.27 1.27)) hide)
     )
+    (property "CatNo" "WM50000-02-ND" (at 267.335 95.885 0)
+      (effects (font (size 1.27 1.27)) hide)
+    )
+    (property "MfgNo" "0416710001" (at 267.335 95.885 0)
+      (effects (font (size 1.27 1.27)) hide)
+    )
     (pin "1")
     (pin "2")
@@
       (effects (font (size 1.27 1.27)) hide)
     )
-    (property "Datasheet" "http://cdn-reichelt.de/documents/datenblatt/B400/OSZI.pdf" (at 31.115 51.435 0)
+    (property "Datasheet" "https://ecsxtal.com/store/pdf/ecs_2100.pdf" (at 31.115 51.435 0)
+      (effects (font (size 1.27 1.27)) hide)
+    )
+    (property "CatNo" "XC235-ND" (at 33.655 51.435 0)
+      (effects (font (size 1.27 1.27)) hide)
+    )
+    (property "MfgNo" "XC235-ND" (at 33.655 51.435 0)
       (effects (font (size 1.27 1.27)) hide)
     )
@@
       (effects (font (size 1.27 1.27)) hide)
     )
-    (property "Datasheet" "~" (at 106.68 189.23 0)
+    (property "Datasheet" "https://www.molex.com/pdm_docs/sd/416710001_sd.pdf" (at 106.68 189.23 0)
+      (effects (font (size 1.27 1.27)) hide)
+    )
+    (property "CatNo" "WM50000-02-ND" (at 106.68 189.23 0)
+      (effects (font (size 1.27 1.27)) hide)
+    )
+    (property "MfgNo" "0416710001" (at 106.68 189.23 0)
       (effects (font (size 1.27 1.27)) hide)
     )
@@
     )
     (property "Datasheet" "http://ww1.microchip.com/downloads/en/DeviceDoc/doc8183.pdf" (at 34.925 113.665 0)
+      (effects (font (size 1.27 1.27)) hide)
+    )
+    (property "CatNo" "ATTINY84A-PU-ND" (at 34.925 113.665 0)
+      (effects (font (size 1.27 1.27)) hide)
+    )
+    (property "MfgNo" "ATTINY84A-PU" (at 34.925 113.665 0)
       (effects (font (size 1.27 1.27)) hide)
     )
@@
       (effects (font (size 1.27 1.27)) hide)
     )
-    (property "Datasheet" "~" (at 151.13 27.305 0)
+    (property "Datasheet" "https://www.molex.com/pdm_docs/sd/416710001_sd.pdf" (at 151.13 27.305 0)
+      (effects (font (size 1.27 1.27)) hide)
+    )
+    (property "CatNo" "WM50000-02-ND" (at 151.13 27.305 0)
+      (effects (font (size 1.27 1.27)) hide)
+    )
+    (property "MfgNo" "0416710001" (at 151.13 27.305 0)
       (effects (font (size 1.27 1.27)) hide)
     )
@@
     )
     (property "Datasheet" "~" (at 77.47 81.915 0)
+      (effects (font (size 1.27 1.27)) hide)
+    )
+    (property "CatNo" "399-C321C104Z5U5TA-ND" (at 77.47 81.915 0)
+      (effects (font (size 1.27 1.27)) hide)
+    )
+    (property "MfgNo" "C321C104Z5U5TA" (at 77.47 81.915 0)
       (effects (font (size 1.27 1.27)) hide)
     )
@@
       (effects (font (size 1.27 1.27)) hide)
     )
+    (property "CatNo" "399-C321C104Z5U5TA-ND" (at 44.45 83.185 0)
+      (effects (font (size 1.27 1.27)) hide)
+    )
+    (property "MfgNo" "C321C104Z5U5TA" (at 44.45 83.185 0)
+      (effects (font (size 1.27 1.27)) hide)
+    )

Commit message: silkscreen and minor tweaks
Parts:
- RV1: CatNo 693-14910F0GJSX10104KA-ND -> 3266Y-1-104LF-ND
Changed lines of the file:
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@@
       (effects (font (size 1.27 1.27)) hide)
     )
-    (property "CatNo" "693-14910F0GJSX10104KA-ND" (at 135.255 128.27 90)
+    (property "CatNo" "3266Y-1-104LF-ND" (at 135.255 128.27 90)
       (effects (font (size 1.27 1.27)))
     )
